File: hardware/radiator_booster.kicad_sch (KiCad schematic)
At the start: 9 parts

Commit message: Finished the pcb layout
Parts:
- removed TP101: 5V, TestPoint:TestPoint_Pad_D1.0mm, symbol Connector:TestPoint_Small
- removed TP102: 3.3V, TestPoint:TestPoint_Pad_D1.0mm, symbol Connector:TestPoint_Small
- removed TP103: I2C_DATA, TestPoint:TestPoint_Pad_D1.0mm, symbol Connector:TestPoint_Small
- removed TP104: I2C_CLK, TestPoint:TestPoint_Pad_D1.0mm, symbol Connector:TestPoint_Small
- removed TP105: FAN_ALERT, TestPoint:TestPoint_Pad_D1.0mm, symbol Connector:TestPoint_Small
- H101, H102, H103, H104: now left out of the parts list
Other:
- note removed: "Test Points"

Commit message: release: v0.1
Other:
- company: (none) -> LP
Changed lines of the file:
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@@
 	(title_block
 		(title "Radiator Booster")
-		(rev "1")
-		(comment 1 "Design for JLCPCB Service")
+		(date "2025-01-19")
+		(rev "0.1")
+		(company "LP")
 	)
 	(junction

Commit message: Finished layout for rev 0.2
Parts:
- removed H101, H102, H103, H104: GND, MountingHole:MountingHole_2.7mm_M2.5_ISO14580_Pad, symbol Mechanical:MountingHole_Pad
Other:
- note removed: "Mounting Holes (M3)"
