File: hardware/radiator_booster.kicad_pcb (KiCad board)
At the start: 4 copper layers, 31 parts, among them J201 USB_C_Receptacle_USB2.0, SW201 RESET, SW202 BOOTSEL, U201 ESP32-C3, U202 USBLC6-2SC6, Y201 40 MHz

Commit message: WIP pcb layout
Parts:
- removed C212, C213: 100n, Capacitor_SMD:C_0402_1005Metric
- removed L202: CMF3216F-900-2P-T, lzptr:CMC-1206
- removed L203: 2n2, Inductor_SMD:L_0402_1005Metric
- added C201: 100n, Capacitor_SMD:C_0402_1005Metric, F.Cu at (126.5, 110.7)
- added C202: 100n, Capacitor_SMD:C_0402_1005Metric, F.Cu at (127.7, 110.7)
- added C203: 10u, Capacitor_SMD:C_0603_1608Metric, F.Cu at (130.6, 111.2)
- added C204: 100n, Capacitor_SMD:C_0402_1005Metric, F.Cu at (133.2, 107.5)
- added C205: 10u, Capacitor_SMD:C_0603_1608Metric, F.Cu at (130.6, 105.2)
- added C302: 3p, Capacitor_SMD:C_0402_1005Metric, F.Cu at (122.2, 91.5)
- added C304: 3p, Capacitor_SMD:C_0402_1005Metric, F.Cu at (122.2, 94.5)
- added C401: 100n, Capacitor_SMD:C_0402_1005Metric, F.Cu at (110.0, 96.5)
- added D201: 3.3V, LED_SMD:LED_0603_1608Metric, F.Cu at (134.8, 122.4)
- added H101: GND, MountingHole:MountingHole_2.7mm_M2.5_ISO14580_Pad, F.Cu at (78.8, 73.2)
- added H102: GND, MountingHole:MountingHole_2.7mm_M2.5_ISO14580_Pad, F.Cu at (144.5, 71.5)
- added H103: GND, MountingHole:MountingHole_2.7mm_M2.5_ISO14580_Pad, F.Cu at (79.6, 128.9)
- added H104: GND, MountingHole:MountingHole_2.7mm_M2.5_ISO14580_Pad, F.Cu at (146.5, 129.2)
- added J401: Fan1, Connector:FanPinHeader_1x04_P2.54mm_Vertical, F.Cu at (92.5, 115.0)
- added J402: Fan2, Connector:FanPinHeader_1x04_P2.54mm_Vertical, F.Cu at (92.3, 106.8)
- added J403: Fan3, Connector:FanPinHeader_1x04_P2.54mm_Vertical, F.Cu at (92.2, 98.8)
- added J404: Fan4, Connector:FanPinHeader_1x04_P2.54mm_Vertical, F.Cu at (92.2, 90.8)
- added J405: Fan5, Connector:FanPinHeader_1x04_P2.54mm_Vertical, F.Cu at (92.2, 82.3)
- added L201: 2n2, Inductor_SMD:L_0402_1005Metric, F.Cu at (127.1, 112.2)
- added L301: 2n2, Inductor_SMD:L_0402_1005Metric, F.Cu at (121.8, 93.0)
- added R201: 1k, Resistor_SMD:R_0402_1005Metric, F.Cu at (136.2, 122.7)
- added R401: 10k, Resistor_SMD:R_0402_1005Metric, F.Cu at (101.9, 111.9)
- added R402: 10k, Resistor_SMD:R_0402_1005Metric, F.Cu at (110.0, 95.4)
- added R403: 2k2, Resistor_SMD:R_0402_1005Metric, F.Cu at (111.7, 101.5)
- added R404: 2k2, Resistor_SMD:R_0402_1005Metric, F.Cu at (111.7, 99.5)
- added R405: 2k2, Resistor_SMD:R_0402_1005Metric, F.Cu at (99.0, 107.9)
- added R406: 2k2, Resistor_SMD:R_0402_1005Metric, F.Cu at (99.0, 109.9)
- added R407: 2k2, Resistor_SMD:R_0402_1005Metric, F.Cu at (99.0, 111.9)
- added R408: 2k2, Resistor_SMD:R_0402_1005Metric, F.Cu at (101.9, 107.9)
- added R409: 2k2, Resistor_SMD:R_0402_1005Metric, F.Cu at (101.9, 109.9)
- added TP101: 5V, TestPoint:TestPoint_Pad_D1.0mm, F.Cu at (139.2, 105.5)
- added TP102: 3.3V, TestPoint:TestPoint_Pad_D1.0mm, F.Cu at (139.2, 108.5)
- added TP103: I2C_DATA, TestPoint:TestPoint_Pad_D1.0mm, F.Cu at (139.2, 111.6)
- added TP104: I2C_CLK, TestPoint:TestPoint_Pad_D1.0mm, F.Cu at (139.2, 114.7)
- added TP105: FAN_ALERT, TestPoint:TestPoint_Pad_D1.0mm, F.Cu at (139.2, 117.7)
- added U201: SPX3819M5-L-3-3, Package_TO_SOT_SMD:SOT-23-5, F.Cu at (130.8, 108.2)
- added U401: EMC2305-1-AP-TR, Package_DFN_QFN:QFN-16-1EP_4x4mm_P0.65mm_EP2.1x2.1mm, F.Cu at (107.3, 99.9)
- C305: renamed from C203; value 10n -> 10u; footprint Capacitor_SMD:C_0402_1005Metric -> Capacitor_SMD:C_0603_1608Metric
- C312: renamed from C209; value 10n -> 10u; footprint Capacitor_SMD:C_0402_1005Metric -> Capacitor_SMD:C_0603_1608Metric
- SW302: renamed from SW202; value BOOTSEL -> BOOT
- moved J301 62.1 mm to (120.0, 120.0)
- moved R301 59.5 mm to (113.0, 114.1), turned to 180 degrees
- moved U302 56.2 mm to (120.0, 100.0), turned to -90 degrees
- moved SW302 50.0 mm to (112.1, 117.8), turned to -90 degrees
- moved R305 47.3 mm to (114.9, 102.0)
- moved R302 46.9 mm to (128.9, 114.2)
- moved R308 46.8 mm to (140.5, 122.9), turned to 90 degrees
- moved R306 46.8 mm to (114.9, 103.0)
- moved U301 46.5 mm to (120.5, 111.2), turned to 90 degrees
- moved D301 44.5 mm to (139.1, 122.4), turned to 90 degrees
- moved R304 41.7 mm to (117.5, 93.0), turned to -90 degrees
- moved R307 38.4 mm to (116.5, 93.0), turned to 90 degrees
- moved SW301 36.8 mm to (128.0, 117.7), turned to -90 degrees
- moved L302 36.4 mm to (120.5, 93.0), turned to -90 degrees
- moved R303 35.0 mm to (125.0, 99.2), turned to 180 degrees
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- renumbered C201 to C301, C202 to C303, C211 to C306, C204 to C307, C205 to C308, C206 to C309, C207 to C310, C208 to C311, C210 to C313, D201 to D301, J201 to J301, L201 to L302, R206 to R301, R207 to R302, R201 to R303, R203 to R304, R204 to R305, R205 to R306, R202 to R307, R208 to R308, SW201 to SW301, U202 to U301, U201 to U302, Y201 to Y301
Connections:
- net /[2] MCU/BOOT renamed /[3] MCU/BOOT
- net /[2] MCU/CHIP_EN renamed /[3] MCU/CHIP_EN
- net /[2] MCU/USB_CONN_CC1 renamed /[3] MCU/USB_CONN_CC1
- net /[2] MCU/USB_CONN_CC2 renamed /[3] MCU/USB_CONN_CC2
- net /[2] MCU/USB_CONN_D+ renamed /[3] MCU/USB_CONN_D+
- net /[2] MCU/USB_CONN_D- renamed /[3] MCU/USB_CONN_D-
- net /[2] MCU/XTAL_IN renamed /[3] MCU/XTAL_IN
- net /[2] MCU/XTAL_N renamed /[3] MCU/XTAL_N
- net /[2] MCU/XTAL_P renamed /[3] MCU/XTAL_P
- net Net-(U201-GPIO2/ADC1_CH2) renamed /[3] MCU/GP2
- net Net-(U201-GPIO8) renamed /[3] MCU/GP8
- D301 pad 2: unconnected-(D201-A-Pad2) -> /[3] MCU/ACT
- J301 pad A8: (no net) -> unconnected-(J301-SBU1-PadA8)
- J301 pad B8: (no net) -> unconnected-(J301-SBU2-PadB8)
- R304 pad 1: +3V3 -> +3.3V
- R305 pad 1: +3V3 -> +3.3V
- R306 pad 1: +3V3 -> +3.3V
- R307 pad 2: +3V3 -> +3.3V
- U301 pad 4: /[2] MCU/USB_CMC_D+ -> /[3] MCU/USB_D+
- U301 pad 6: /[2] MCU/USB_CMC_D- -> /[3] MCU/USB_D-
- U302 pad 1: unconnected-(U201-LNA_IN-Pad1) -> /[3] MCU/LNA_IN
- U302 pad 13: unconnected-(U201-MTDO/GPIO7-Pad13) -> /FAN_ALERT
- U302 pad 16: unconnected-(U201-GPIO10-Pad16) -> /[3] MCU/ACT
- U302 pad 25: /[2] MCU/USB_D- -> /[3] MCU/USB_D-
- U302 pad 26: /[2] MCU/USB_D+ -> /[3] MCU/USB_D+
- U302 pad 8: unconnected-(U201-GPIO3/ADC1_CH3-Pad8) -> /I2C_CLK
- U302 pad 9: unconnected-(U201-MTMS/GPIO4/ADC1_CH4-Pad9) -> /I2C_DATA
Other:
- board text added: "3.3V"
- board text added: "ACT"

Commit message: Finished the pcb layout
Parts:
- removed TP101: 5V, TestPoint:TestPoint_Pad_D1.0mm
- removed TP102: 3.3V, TestPoint:TestPoint_Pad_D1.0mm
- removed TP103: I2C_DATA, TestPoint:TestPoint_Pad_D1.0mm
- removed TP104: I2C_CLK, TestPoint:TestPoint_Pad_D1.0mm
- removed TP105: FAN_ALERT, TestPoint:TestPoint_Pad_D1.0mm
- added AE301: Antenna, lzptr:ANT5320LL45R2400A, F.Cu at (172.0, 65.7)
- U302: value ESP32-C3 -> ESP32-C3FH4
- moved J404 101.4 mm to (192.6, 76.0)
- moved J405 100.4 mm to (192.6, 84.0)
- moved J401 68.3 mm to (148.6, 76.0)
- moved H103 67.6 mm to (142.0, 103.0)
- moved H101 63.6 mm to (142.0, 66.0)
- moved R405 63.3 mm to (155.2, 78.9), turned to 180 degrees
- moved R409 61.1 mm to (158.9, 87.9), turned to 90 degrees
- moved J402 60.8 mm to (148.6, 84.0)
- moved R406 60.1 mm to (151.7, 81.1)
- moved R407 59.8 mm to (151.7, 83.7)
- moved R401 58.2 mm to (154.9, 87.9), turned to -90 degrees
- moved R408 58.0 mm to (156.3, 87.9), turned to 90 degrees
- moved J403 56.8 mm to (148.6, 92.0)
- moved R301 53.8 mm to (164.6, 98.9), turned to 90 degrees
- moved C202 53.5 mm to (178.9, 95.4)
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Routing:
- net +5V: track 0.00 -> 112.1 mm, vias 0 -> 1
- net +3.3V: track 0.00 -> 96.1 mm, vias 0 -> 9
- net /[3] MCU/CHIP_EN: track 0.00 -> 70.1 mm, vias 0 -> 2
- net /[4] Fan Control/PWM4: track 0.00 -> 62.3 mm, vias 0 -> 1
- net /[4] Fan Control/TACH4: track 0.00 -> 58.9 mm, vias 0 -> 1
- net /[4] Fan Control/PWM5: track 0.00 -> 46.4 mm, vias 0 -> 1
- net /[4] Fan Control/TACH5: track 0.00 -> 44.7 mm, vias 0 -> 1
- net /[3] MCU/ACT: track 0.00 -> 34.0 mm
- net GND: track 0.00 -> 33.0 mm, vias 0 -> 147
- net /[3] MCU/BOOT: track 0.00 -> 26.9 mm
- net /FAN_ALERT: track 0.00 -> 24.5 mm, vias 0 -> 2
- net VBUS: track 0.00 -> 24.0 mm
- net /[4] Fan Control/TACH3: track 0.00 -> 23.5 mm, vias 0 -> 1
- net /[4] Fan Control/TACH2: track 0.00 -> 18.9 mm
- net /[4] Fan Control/Tach1: track 0.00 -> 17.0 mm
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- added copper zone on B.Cu, net +3.3V
- added copper zone on F.Cu, net +3.3V
- added copper zone on F.Cu, net GND
- added copper zone on In1.Cu, net GND
- added copper zone on In2.Cu, net GND
Other:
- board outline added: 58 x 47 mm
- board text added: "FAN 1"
- board text added: "FAN 2"
- board text added: "FAN 3"
- board text added: "FAN 4"
- board text added: "FAN 5"

Commit message: release: v0.1
Parts:
- AE301: footprint lzptr:ANT5320LL45R2400A -> lzptr:Rainsun-AN9520-245
- D201, D301: footprint LED_SMD:LED_0603_1608Metric -> LED_SMD:LED_0805_2012Metric
- moved AE301 5.51 mm to (176.8, 63.0), turned to 0 degrees
- moved R305 2.33 mm to (164.8, 85.6), turned to 90 degrees
- moved R307 1.31 mm to (165.0, 77.2)
- moved C313 1.28 mm to (164.5, 75.6)
- moved R306 0.80 mm to (163.7, 89.3), turned to -90 degrees
- moved D301 0.25 mm to (154.8, 104.0)
- moved D201 0.20 mm to (150.5, 104.0)
Routing:
- net +3.3V: track 96.1 -> 89.5 mm, vias 9 -> 11
- net Net-(AE301-A): track 8.58 -> 13.8 mm
- net /[3] MCU/GP8: track 6.23 -> 3.05 mm
- net /[3] MCU/CHIP_EN: track 70.1 -> 72.2 mm
- net /[3] MCU/BOOT: track 26.9 -> 26.1 mm
- net /FAN_ALERT: track 24.5 -> 25.0 mm
- net GND: vias 147 -> 145
Other:
- board text added: "LP 01/25 REV 0.1"
- board text added: "Radiator Booster"

Commit message: Fixed routing at intel pwm fan connectors
Connections:
- net /[3] MCU/LNA_IN renamed /[3] MCU/RF_IN
- net Net-(AE301-A) renamed /[3] MCU/RF_ANT
- J401 pad 2: /[4] Fan Control/PWM1 -> unconnected-(J401-Pin_2-Pad2)
- J401 pad 3: /[4] Fan Control/Tach1 -> unconnected-(J401-Pin_3-Pad3)
- J401 pad 4: +5V -> /[4] Fan Control/PWM1
- J402 pad 2: /[4] Fan Control/PWM2 -> unconnected-(J402-Pin_2-Pad2)
- J402 pad 3: /[4] Fan Control/TACH2 -> unconnected-(J402-Pin_3-Pad3)
- J402 pad 4: +5V -> /[4] Fan Control/PWM2
- J403 pad 2: /[4] Fan Control/PWM3 -> unconnected-(J403-Pin_2-Pad2)
- J403 pad 3: /[4] Fan Control/TACH3 -> unconnected-(J403-Pin_3-Pad3)
- J403 pad 4: +5V -> /[4] Fan Control/PWM3
- J404 pad 2: /[4] Fan Control/PWM4 -> unconnected-(J404-Pin_2-Pad2)
- J404 pad 3: /[4] Fan Control/TACH4 -> unconnected-(J404-Pin_3-Pad3)
- J404 pad 4: +5V -> /[4] Fan Control/PWM4
- J405 pad 2: /[4] Fan Control/PWM5 -> unconnected-(J405-Pin_2-Pad2)
- J405 pad 3: /[4] Fan Control/TACH5 -> unconnected-(J405-Pin_3-Pad3)
- J405 pad 4: +5V -> unconnected-(J405-Pin_4-Pad4)

Commit message: Finished layout for rev 0.2
Parts:
- removed H101, H102, H103, H104: GND, MountingHole:MountingHole_2.7mm_M2.5_ISO14580_Pad
- AE301: value Antenna -> ANT3216LL00R2400A; footprint lzptr:Rainsun-AN9520-245 -> lzptr:ANT3216LL00R2400A
- moved J404 47.5 mm to (147.9, 92.2)
- moved J405 47.5 mm to (147.9, 100.2)
- moved U201 25.9 mm to (156.1, 89.5)
- moved C204 25.9 mm to (158.5, 88.8)
- moved C205 25.9 mm to (155.9, 86.5)
- moved C203 25.5 mm to (156.3, 92.5), turned to 180 degrees
- moved C202 21.0 mm to (158.5, 90.8)
- moved L201 19.1 mm to (159.4, 92.6), turned to 180 degrees
- moved C201 17.3 mm to (160.4, 90.8)
- moved R409 15.0 mm to (150.4, 100.2)
- moved R405 11.6 mm to (150.4, 68.3), turned to 90 degrees
- moved Y301 9.51 mm to (171.6, 87.7)
- moved C303 9.21 mm to (170.8, 90.3), turned to 180 degrees
- moved R401 9.11 mm to (162.0, 82.2), turned to 180 degrees
- moved R201 8.04 mm to (154.2, 96.8), turned to 180 degrees
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Connections:
- J401 pad 2: unconnected-(J401-Pin_2-Pad2) -> +5V
- J401 pad 3: unconnected-(J401-Pin_3-Pad3) -> /[4] Fan Control/TACH1
- J402 pad 2: unconnected-(J402-Pin_2-Pad2) -> +5V
- J402 pad 3: unconnected-(J402-Pin_3-Pad3) -> /[4] Fan Control/TACH2
- J403 pad 2: unconnected-(J403-Pin_2-Pad2) -> +5V
- J403 pad 3: unconnected-(J403-Pin_3-Pad3) -> /[4] Fan Control/TACH3
- J404 pad 2: unconnected-(J404-Pin_2-Pad2) -> +5V
- J404 pad 3: unconnected-(J404-Pin_3-Pad3) -> /[4] Fan Control/TACH4
- J405 pad 2: unconnected-(J405-Pin_2-Pad2) -> +5V
- J405 pad 3: unconnected-(J405-Pin_3-Pad3) -> /[4] Fan Control/TACH5
- J405 pad 4: unconnected-(J405-Pin_4-Pad4) -> /[4] Fan Control/PWM5
- R405 pad 2: /[4] Fan Control/Tach1 -> /[4] Fan Control/TACH1
- U401 pad 6: /[4] Fan Control/Tach1 -> /[4] Fan Control/TACH1
Routing:
- net +5V: track 112.1 -> 54.5 mm, vias 1 -> 2
- net +3.3V: track 89.5 -> 132.4 mm, vias 11 -> 9
- net /[4] Fan Control/PWM4: track 62.3 -> 19.9 mm
- net /[4] Fan Control/TACH4: track 58.9 -> 21.1 mm
- net /[3] MCU/CHIP_EN: track 72.2 -> 36.0 mm
- net /[4] Fan Control/TACH1: track 0.00 -> 25.0 mm
- net GND: track 33.0 -> 13.2 mm, vias 145 -> 251
- net /[4] Fan Control/PWM5: track 46.4 -> 29.1 mm
- net /[4] Fan Control/Tach1: track 17.0 -> 0.00 mm
- net /[4] Fan Control/TACH5: track 44.7 -> 29.6 mm
- net /[4] Fan Control/PWM1: track 15.0 -> 27.6 mm, vias 1 -> 0
- net /[3] MCU/XTAL_P: track 2.18 -> 14.0 mm
- net /[3] MCU/RF_ANT: track 13.8 -> 4.29 mm
- net /FAN_ALERT: track 25.0 -> 17.9 mm
- net /[4] Fan Control/TACH3: track 23.5 -> 16.4 mm
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- added copper zone on B.Cu, net GND
- removed copper zone on B.Cu, net +3.3V
- removed copper zone on F.Cu, net +3.3V
Other:
- board size 58 x 47 mm -> 40 x 40 mm
- board text added: "LP 03/25 REV 0.2"
- board text removed: "LP 01/25 REV 0.1"

Commit message: Final touches
Other:
- board text added: "Radiator Booster LP 03/25 REV 0.2"
- board text added: "↓FAN 4"
- board text added: "↓FAN 5"
- board text removed: "FAN 4"
- board text removed: "FAN 5"
- board text removed: "LP 03/25 REV 0.2"
- board text removed: "Radiator Booster"
Changed lines of the file:
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@@
 		(layer "Edge.Cuts")
 	)
-	(gr_text "FAN 5"
-		(at 202.8 83.15 90)
+	(gr_text "↓FAN 5\n"
+		(at 138.505 96.74 0)
 		(layer "F.SilkS")
 		(effects
@@
 				(size 1 1)
 				(thickness 0.15)
-			)
-			(justify left bottom)
-		)
-	)
-	(gr_text "LP 03/25\nREV 0.2"
-		(at 150.85 62.8 0)
-		(layer "F.SilkS")
-		(effects
-			(font
-				(size 0.5 0.5)
-				(thickness 0.1)
 			)
 			(justify left bottom)
@@
 		)
 	)
-	(gr_text "Radiator Booster"
-		(at 150.7 60.9 0)
-		(layer "F.SilkS")
-		(effects
-			(font
-				(size 1.5 1.5)
-				(thickness 0.1)
-			)
-			(justify left bottom)
-		)
-	)
 	(gr_text "FAN 1\n"
-		(at 124.25 72 90)
+		(at 144.89 72.32 0)
 		(layer "F.SilkS")
 		(effects
@@
 	)
 	(gr_text "FAN 3\n"
-		(at 129.4 98.85 90)
+		(at 144.925 88.23 0)
 		(layer "F.SilkS")
 		(effects
@@
 	)
 	(gr_text "FAN 2\n"
-		(at 124.25 80 90)
+		(at 144.915 80.27 0)
 		(layer "F.SilkS")
 		(effects
@@
 		)
 	)
-	(gr_text "FAN 4"
-		(at 202.8 75.15 90)
+	(gr_text "↓FAN 4"
+		(at 138.505 88.78 0)
 		(layer "F.SilkS")
 		(effects
@@
 			)
 			(justify left bottom)
+		)
+	)
+	(gr_text "Radiator Booster\nLP 03/25\nREV 0.2"
+		(at 157.77 67.89 0)
+		(layer "B.SilkS")
+		(effects
+			(font
+				(size 0.5 0.5)
+				(thickness 0.1)
+			)
+			(justify left bottom mirror)
 		)
 	)
@@
 	)
 	(via
-		(at 150.4 71.25)
+		(at 150.55 71.070003)
 		(size 0.7)
 		(drill 0.3)
@@
 	)
 	(via
-		(at 152.8 69.25)
+		(at 152.95 69.070003)
 		(size 0.7)
 		(drill 0.3)
@@
 	)
 	(via
-		(at 155.2 70.25)
+		(at 155.35 70.070003)
 		(size 0.7)
 		(drill 0.3)
@@
 	)
 	(via
-		(at 152.8 72.25)
-		(size 0.7)
-		(drill 0.3)
-		(layers "F.Cu" "B.Cu")
-		(free yes)
-		(net 1)
-	)
-	(via
-		(at 151.6 70.25)
+		(at 152.95 72.070003)
+		(size 0.7)
+		(drill 0.3)
+		(layers "F.Cu" "B.Cu")
+		(free yes)
+		(net 1)
+	)
+	(via
+		(at 151.75 70.070003)
 		(size 0.7)
 		(drill 0.3)
@@
 	)
 	(via
-		(at 150.4 73.249997)
+		(at 150.55 73.07)
 		(size 0.7)
 		(drill 0.3)
@@
 	)
 	(via
-		(at 151.6 69.25)
+		(at 151.75 69.070003)
 		(size 0.7)
 		(drill 0.3)
@@
 	)
 	(via
-		(at 152.8 73.249997)
+		(at 152.95 73.07)
 		(size 0.7)
 		(drill 0.3)
@@
 	)
 	(via
-		(at 155.2 72.25)
+		(at 155.35 72.070003)
 		(size 0.7)
 		(drill 0.3)
@@
 	)
 	(via
-		(at 152.8 71.25)
+		(at 152.95 71.070003)
 		(size 0.7)
 		(drill 0.3)
@@
 	)
 	(via
-		(at 151.6 71.25)
+		(at 151.75 71.070003)
 		(size 0.7)
 		(drill 0.3)
@@
 	)
 	(via
-		(at 152.8 70.25)
+		(at 152.95 70.070003)
 		(size 0.7)
 		(drill 0.3)
@@
 	)
 	(via
-		(at 155.2 69.25)
+		(at 155.35 69.070003)
 		(size 0.7)
 		(drill 0.3)
@@
 	)
 	(via
-		(at 154 73.249997)
+		(at 154.15 73.07)
 		(size 0.7)
 		(drill 0.3)
@@
 	)
 	(via
-		(at 154 69.25)
+		(at 154.15 69.070003)
 		(size 0.7)
 		(drill 0.3)
@@
 	)
 	(via
-		(at 155.2 73.249997)
+		(at 155.35 73.07)
 		(size 0.7)
 		(drill 0.3)
@@
 	)
 	(via
-		(at 150.4 72.25)
+		(at 150.55 72.070003)
 		(size 0.7)
 		(drill 0.3)
@@
 	)
 	(via
-		(at 154 72.25)
+		(at 154.15 72.070003)
 		(size 0.7)
 		(drill 0.3)
@@
 	)
 	(via
-		(at 150.4 70.25)
+		(at 150.55 70.070003)
 		(size 0.7)
 		(drill 0.3)
@@
 	)
 	(via
-		(at 151.6 72.25)
+		(at 151.75 72.070003)
 		(size 0.7)
 		(drill 0.3)
@@
 	)
 	(via
-		(at 155.2 71.25)
+		(at 155.35 71.070003)
 		(size 0.7)
 		(drill 0.3)
@@
 	)
 	(via
-		(at 154 70.25)
+		(at 154.15 70.070003)
 		(size 0.7)
 		(drill 0.3)
@@
 	)
 	(via
-		(at 154 71.25)
-		(size 0.7)
-		(drill 0.3)
-		(layers "F.Cu" "B.Cu")
-		(free yes)
-		(net 1)
-	)
-	(via
-		(at 151.6 73.249997)
-		(size 0.7)
-		(drill 0.3)
+		(at 154.15 71.070003)
+		(size 0.7)
+		(drill 0.3)
+		(layers "F.Cu" "B.Cu")
+		(free yes)
+		(net 1)
+	)
+	(via
+		(at 151.75 73.07)
+		(size 0.7)
+		(drill 0.3)

Commit message: Added production files
Parts:
- moved C205 0.07 mm to (155.9, 86.4)
Routing:
- net GND: vias 251 -> 212
