File: hardware/fan_control.kicad_sch (KiCad schematic)
At the start: 16 parts, among them J401 Fan1, J402 Fan2, J403 Fan3, J404 Fan4, J405 Fan5, U401 EMC2305-1-AP-TR

Commit message: WIP pcb layout
Parts:
- renumbered R409 to R401, R401 to R402, R402 to R403, R403 to R404, R404 to R405, R405 to R406, R406 to R407, R407 to R408, R408 to R409
Connections:
- net TACH3: now reaches J403.3 (Pin_3), R407.2, U401.10 (TACH3)
- net PWM4: now reaches J404.2 (Pin_2), U401.13 (PWM4)
- net TACH4: now reaches J404.3 (Pin_3), R408.2, U401.14 (TACH4)
- net PWM5: now reaches J405.2 (Pin_2), U401.15 (PWM5)
- net TACH5: now reaches J405.3 (Pin_3), R409.2, U401.16 (TACH5)
- net ADDR_SEL: now reaches R402.1, U401.4 (ADDR_SEL)
- net PWM1: now reaches J401.2 (Pin_2), U401.5 (PWM1)
- net Tach1: now reaches J401.3 (Pin_3), R405.2, U401.6 (TACH1)
- net PWM2: now reaches J402.2 (Pin_2), U401.7 (PWM2)
- net TACH2: now reaches J402.3 (Pin_3), R406.2, U401.8 (TACH2)
- net PWM3: now reaches J403.2 (Pin_2), U401.9 (PWM3)
Changed lines of the file:
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@@
+		)
+	)
+	(label "TACH2"
+		(at 113.03 69.85 0)
+		(fields_autoplaced yes)
+		(effects
+			(font
+				(size 1.27 1.27)
+			)
+			(justify left bottom)
+		)
+	)
+	(label "TACH5"
+		(at 113.03 88.9 0)
+		(fields_autoplaced yes)
+		(effects
+			(font
+				(size 1.27 1.27)
+			)
+			(justify left bottom)
+		)
+	)
+	(label "PWM5"
+		(at 113.03 86.36 0)
+		(fields_autoplaced yes)
+		(effects
+			(font
+				(size 1.27 1.27)
+			)
+			(justify left bottom)
+		)
+	)
+	(label "TACH4"
+		(at 113.03 82.55 0)
+		(fields_autoplaced yes)
+		(effects
+			(font
+				(size 1.27 1.27)
+			)
+			(justify left bottom)
+		)
+	)
+	(label "PWM4"
+		(at 113.03 80.01 0)
+		(fields_autoplaced yes)
+		(effects
+			(font
+				(size 1.27 1.27)
+			)
+			(justify left bottom)
+		)
+	)
+	(label "PWM2"
+		(at 113.03 67.31 0)
+		(fields_autoplaced yes)
+		(effects
+			(font
+				(size 1.27 1.27)
+			)
+			(justify left bottom)
+		)
+	)
+	(label "Tach1"
+		(at 113.03 63.5 0)
+		(fields_autoplaced yes)
+		(effects
+			(font
+				(size 1.27 1.27)
+			)
+			(justify left bottom)
+		)
+	)
+	(label "TACH3"
+		(at 113.03 76.2 0)
+		(fields_autoplaced yes)
+		(effects
+			(font
+				(size 1.27 1.27)
+			)
+			(justify left bottom)
+		)
+	)
+	(label "PWM3"
+		(at 113.03 73.66 0)
+		(fields_autoplaced yes)
+		(effects
+			(font
+				(size 1.27 1.27)
+			)
+			(justify left bottom)
+		)
+	)
+	(label "ADDR_SEL"
+		(at 69.85 66.04 0)
+		(fields_autoplaced yes)
+		(effects
+			(font
+				(size 1.27 1.27)
+			)
+			(justify left bottom)
+		)
+	)
+	(label "PWM1"
+		(at 113.03 60.96 0)
+		(fields_autoplaced yes)
+		(effects
+			(font
+				(size 1.27 1.27)
+			)
+			(justify left bottom)
 		)
 	)
@@
 		(on_board yes)
 		(dnp no)
-		(property "Reference" "#PWR0409"
+		(property "Reference" "#PWR0401"
 			(at 41.91 57.15 0)
 			(effects
@@
 			(project "radiator_booster"
 				(path "/af3170cb-38e8-4f1f-8d67-3c2d4410beea/25b872c9-4a13-434a-a096-25f68f332965"
-					(reference "#PWR0409")
+					(reference "#PWR0401")
 					(unit 1)
 				)
@@
 		(on_board yes)
 		(dnp no)
-		(property "Reference" "R409"
+		(property "Reference" "R401"
 			(at 34.798 57.658 0)
 			(effects
@@
 			(project "radiator_booster"
 				(path "/af3170cb-38e8-4f1f-8d67-3c2d4410beea/25b872c9-4a13-434a-a096-25f68f332965"
-					(reference "R409")
+					(reference "R401")
 					(unit 1)
 				)
@@
 		(on_board yes)
 		(dnp no)
-		(property "Reference" "#PWR0401"
+		(property "Reference" "#PWR0405"
 			(at 96.52 41.91 0)
 			(effects
@@
 			(project "radiator_booster"
 				(path "/af3170cb-38e8-4f1f-8d67-3c2d4410beea/25b872c9-4a13-434a-a096-25f68f332965"
-					(reference "#PWR0401")
+					(reference "#PWR0405")
 					(unit 1)
 				)
@@
 		(on_board yes)
 		(dnp no)
-		(property "Reference" "#PWR0408"
+		(property "Reference" "#PWR0407"
 			(at 124.46 44.45 0)
 			(effects
@@
 			(project "radiator_booster"
 				(path "/af3170cb-38e8-4f1f-8d67-3c2d4410beea/25b872c9-4a13-434a-a096-25f68f332965"
-					(reference "#PWR0408")
+					(reference "#PWR0407")
 					(unit 1)
 				)
@@
 		(on_board yes)
 		(dnp no)
-		(property "Reference" "R403"
+		(property "Reference" "R404"
 			(at 77.47 50.292 0)
 			(effects
@@
 			(project "radiator_booster"
 				(path "/af3170cb-38e8-4f1f-8d67-3c2d4410beea/25b872c9-4a13-434a-a096-25f68f332965"
-					(reference "R403")
+					(reference "R404")
 					(unit 1)
 				)
@@
 		(dnp no)
 		(fields_autoplaced yes)
-		(property "Reference" "#PWR0405"
+		(property "Reference" "#PWR0408"
 			(at 168.91 54.61 0)
 			(effects
@@
 			(project "radiator_booster"
 				(path "/af3170cb-38e8-4f1f-8d67-3c2d4410beea/25b872c9-4a13-434a-a096-25f68f332965"
-					(reference "#PWR0405")
+					(reference "#PWR0408")
 					(unit 1)
 				)
@@
 		(dnp no)
 		(fields_autoplaced yes)
-		(property "Reference" "#PWR0406"
+		(property "Reference" "#PWR0409"
 			(at 171.45 128.27 0)
 			(effects
@@
 			(project "radiator_booster"
 				(path "/af3170cb-38e8-4f1f-8d67-3c2d4410beea/25b872c9-4a13-434a-a096-25f68f332965"
-					(reference "#PWR0406")
+					(reference "#PWR0409")
 					(unit 1)
 				)
@@
 		(on_board yes)
 		(dnp no)
-		(property "Reference" "R405"
+		(property "Reference" "R406"
 			(at 130.81 49.022 0)
 			(effects
@@
 			(project "radiator_booster"
 				(path "/af3170cb-38e8-4f1f-8d67-3c2d4410beea/25b872c9-4a13-434a-a096-25f68f332965"
-					(reference "R405")
+					(reference "R406")
 					(unit 1)
 				)
@@
 		(on_board yes)
 		(dnp no)
-		(property "Reference" "R408"
+		(property "Reference" "R409"
 			(at 153.67 49.022 0)
 			(effects
@@
 			(project "radiator_booster"
 				(path "/af3170cb-38e8-4f1f-8d67-3c2d4410beea/25b872c9-4a13-434a-a096-25f68f332965"
-					(reference "R408")
+					(reference "R409")
 					(unit 1)
 				)
@@
 		(on_board yes)
 		(dnp no)
-		(property "Reference" "R402"
+		(property "Reference" "R403"
 			(at 68.58 50.292 0)
 			(effects
@@
 			(project "radiator_booster"
 				(path "/af3170cb-38e8-4f1f-8d67-3c2d4410beea/25b872c9-4a13-434a-a096-25f68f332965"
-					(reference "R402")
+					(reference "R403")
 					(unit 1)
 				)
@@
 		(on_board yes)
 		(dnp no)
-		(property "Reference" "R401"
+		(property "Reference" "R402"
 			(at 56.642 57.658 0)
 			(effects
@@
 			(project "radiator_booster"
 				(path "/af3170cb-38e8-4f1f-8d67-3c2d4410beea/25b872c9-4a13-434a-a096-25f68f332965"
-					(reference "R401")
+					(reference "R402")
 					(unit 1)
 				)
@@
 		(dnp no)
 		(fields_autoplaced yes)
-		(property "Reference" "#PWR0403"
+		(property "Reference" "#PWR0406"
 			(at 96.52 102.87 0)
 			(effects
@@
 			(project "radiator_booster"
 				(path "/af3170cb-38e8-4f1f-8d67-3c2d4410beea/25b872c9-4a13-434a-a096-25f68f332965"
-					(reference "#PWR0403")
+					(reference "#PWR0406")
 					(unit 1)
 				)
@@
 		(on_board yes)
 		(dnp no)
-		(property "Reference" "#PWR0407"
+		(property "Reference" "#PWR0403"
 			(at 69.85 45.72 0)
 			(effects
@@
 			(project "radiator_booster"
 				(path "/af3170cb-38e8-4f1f-8d67-3c2d4410beea/25b872c9-4a13-434a-a096-25f68f332965"
-					(reference "#PWR0407")
+					(reference "#PWR0403")
 					(unit 1)
 				)
@@
 		(on_board yes)
 		(dnp no)
-		(property "Reference" "R406"
+		(property "Reference" "R407"
 			(at 138.43 49.022 0)
 			(effects
@@
 			(project "radiator_booster"
 				(path "/af3170cb-38e8-4f1f-8d67-3c2d4410beea/25b872c9-4a13-434a-a096-25f68f332965"
-					(reference "R406")
+					(reference "R407")
 					(unit 1)
 				)
@@
 		(on_board yes)
 		(dnp no)
-		(property "Reference" "R407"
+		(property "Reference" "R408"
 			(at 146.05 49.022 0)
 			(effects
@@
 			(project "radiator_booster"
 				(path "/af3170cb-38e8-4f1f-8d67-3c2d4410beea/25b872c9-4a13-434a-a096-25f68f332965"
-					(reference "R407")
+					(reference "R408")
 					(unit 1)
 				)
@@
 		(on_board yes)
 		(dnp no)
-		(property "Reference" "R404"
+		(property "Reference" "R405"
 			(at 123.19 49.022 0)
 			(effects
@@
 			(project "radiator_booster"
 				(path "/af3170cb-38e8-4f1f-8d67-3c2d4410beea/25b872c9-4a13-434a-a096-25f68f332965"
-					(reference "R404")
-					(unit 1)
-				)
+					(reference "R405")
+					(unit 1)
+				)

Commit message: Finished the pcb layout
Parts:
- J401: Position Offset (none) -> 0,-0.85; Rotation Offset (none) -> 180
- J402, J403, J404, J405: MPN (none) -> C240840; Position Offset (none) -> 0,-0.85; Rotation Offset (none) -> 180
Changed lines of the file:
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@@
+			)
+		)
+		(property "Rotation Offset" "180"
+			(at 179.07 57.15 0)
+			(effects
+				(font
+					(size 1.27 1.27)
+				)
+				(hide yes)
+			)
+		)
+		(property "Position Offset" "0,-0.85"
+			(at 179.07 57.15 0)
+			(effects
+				(font
+					(size 1.27 1.27)
+				)
+				(hide yes)
 			)
 		)
@@
 			)
 		)
+		(property "MPN" "C240840"
+			(at 179.07 114.3 0)
+			(effects
+				(font
+					(size 1.27 1.27)
+				)
+				(hide yes)
+			)
+		)
+		(property "Rotation Offset" "180"
+			(at 179.07 114.3 0)
+			(effects
+				(font
+					(size 1.27 1.27)
+				)
+				(hide yes)
+			)
+		)
+		(property "Position Offset" "0,-0.85"
+			(at 179.07 114.3 0)
+			(effects
+				(font
+					(size 1.27 1.27)
+				)
+				(hide yes)
+			)
+		)
 		(pin "4"
 		)
@@
 			)
 		)
+		(property "MPN" "C240840"
+			(at 179.07 71.12 0)
+			(effects
+				(font
+					(size 1.27 1.27)
+				)
+				(hide yes)
+			)
+		)
+		(property "Rotation Offset" "180"
+			(at 179.07 71.12 0)
+			(effects
+				(font
+					(size 1.27 1.27)
+				)
+				(hide yes)
+			)
+		)
+		(property "Position Offset" "0,-0.85"
+			(at 179.07 71.12 0)
+			(effects
+				(font
+					(size 1.27 1.27)
+				)
+				(hide yes)
+			)
+		)
 		(pin "4"
 		)
@@
 			)
 		)
+		(property "MPN" "C240840"
+			(at 179.07 85.09 0)
+			(effects
+				(font
+					(size 1.27 1.27)
+				)
+				(hide yes)
+			)
+		)
+		(property "Rotation Offset" "180"
+			(at 179.07 85.09 0)
+			(effects
+				(font
+					(size 1.27 1.27)
+				)
+				(hide yes)
+			)
+		)
+		(property "Position Offset" "0,-0.85"
+			(at 179.07 85.09 0)
+			(effects
+				(font
+					(size 1.27 1.27)
+				)
+				(hide yes)
+			)
+		)
 		(pin "4"
 		)
@@
 			(at 179.07 100.33 0)
 			(effects
+				(font
+					(size 1.27 1.27)
+				)
+				(hide yes)
+			)
+		)
+		(property "MPN" "C240840"
+			(at 179.07 100.33 0)
+			(effects
+				(font
+					(size 1.27 1.27)
+				)
+				(hide yes)
+			)
+		)
+		(property "Rotation Offset" "180"
+			(at 179.07 100.33 0)
+			(effects
+				(font
+					(size 1.27 1.27)
+				)
+				(hide yes)
+			)
+		)
+		(property "Position Offset" "0,-0.85"
+			(at 179.07 100.33 0)
+			(effects

Commit message: release: v0.1
Parts:
- R401, R402: MPN C60490 -> C25744
- R403, R404, R405, R406, R407, R408, R409: MPN C326602 -> C25879
- U401: Rotation Offset (none) -> 180
Other:
- company: (none) -> LP
- title: (none) -> Radiator Booster
Changed lines of the file:
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@@
 	(generator_version "8.0")
 	(paper "A4")
+	(title_block
+		(title "Radiator Booster")
+		(date "2025-01-19")
+		(rev "0.1")
+		(company "LP")
+	)
 	(junction
 		(at 154.94 88.9)
@@
 			)
 		)
-		(property "MPN" "C60490"
+		(property "MPN" "C25744"
 			(at 41.91 59.69 0)
 			(effects
@@
 			)
 		)
+		(property "Rotation Offset" "180"
+			(at 96.52 74.93 0)
+			(effects
+				(font
+					(size 1.27 1.27)
+				)
+				(hide yes)
+			)
+		)
 		(pin "3"
 		)
@@
 			)
 		)
-		(property "MPN" "C326602"
+		(property "MPN" "C25879"
 			(at 78.74 52.07 0)
 			(effects
@@
 			)
 		)
-		(property "MPN" "C326602"
+		(property "MPN" "C25879"
 			(at 132.08 50.8 0)
 			(effects
@@
 			)
 		)
-		(property "MPN" "C326602"
+		(property "MPN" "C25879"
 			(at 154.94 50.8 0)
 			(effects
@@
 			)
 		)
-		(property "MPN" "C326602"
+		(property "MPN" "C25879"
 			(at 69.85 52.07 0)
 			(effects
@@
 			)
 		)
-		(property "MPN" "C60490"
+		(property "MPN" "C25744"
 			(at 49.53 59.69 0)
 			(effects
@@
 			)
 		)
-		(property "MPN" "C326602"
+		(property "MPN" "C25879"
 			(at 139.7 50.8 0)
 			(effects
@@
 			)
 		)
-		(property "MPN" "C326602"
+		(property "MPN" "C25879"
 			(at 147.32 50.8 0)
 			(effects
@@
 			)
 		)
-		(property "MPN" "C326602"
+		(property "MPN" "C25879"
 			(at 124.46 50.8 0)
 			(effects

Commit message: Fixed routing at intel pwm fan connectors
Connections:
- net +5V: now also J401.2 (Pin_2), J402.2 (Pin_2), J403.2 (Pin_2), J404.2 (Pin_2), J405.2 (Pin_2); no longer J401.4 (Pin_4), J402.4 (Pin_4), J403.4 (Pin_4), J404.4 (Pin_4), J405.4 (Pin_4)
- net PWM1: now also J401.4 (Pin_4); no longer J401.2 (Pin_2)
- net PWM2: now also J402.4 (Pin_4); no longer J402.2 (Pin_2)
- net PWM3: now also J403.4 (Pin_4); no longer J403.2 (Pin_2)
- net PWM4: now also J404.4 (Pin_4); no longer J404.2 (Pin_2)
- net PWM5: now also J405.4 (Pin_4); no longer J405.2 (Pin_2)
- net Tach1 renamed TACH1
Other:
- moved on the sheet: J401, J402, J403, J404, J405
